Commit message: Add files via upload

File: hardware/SO100arm_7dof/urdf/so100dof7.urdf (robot description, URDF)
Before this commit: robot re-assemble, 10 links, 11 joints
Joints:
- removed joint STS3215_03a-v2_Rigid-15
- removed joint STS3215_03a-v2_Rigid-16
- removed joint STS3215_03a-v2_Rigid-19
- removed joint STS3215_03a-v2_Rigid-2
- removed joint STS3215_03a-v2_Rigid-4
- removed joint STS3215_03a-v2_Rigid-7
- removed joint STS3215_03a-v2_Rigid-9
- added joint STS3215_03a-v2_Revolute-15: type continuous, parent STS3215_03a-v2, child Wrist_Roll_Pitch_08i-v1, origin xyz=-0.02651877752090119 -0.03191000591767831 -0.00899891325538654 rpy=-0.019750555373295158 -0.7852030704405512 -3.1136593337733354, axis 0.500962 0.844217 0.19061599999999998
- added joint STS3215_03a-v2_Revolute-16: type continuous, parent STS3215_03a-v2, child Wrist_Roll_08c-v1-v2, origin xyz=0.012500004374636369 1.1984412395804612e-09 0.018699997382835055 rpy=-1.324799292993419 0.9954112014990447 0.4011360195493793, axis -0.8389830000000003 -0.5277760000000001 0.13251500000000002
- added joint STS3215_03a-v2_Revolute-19: type continuous, parent STS3215_03a-v2, child Moving_Jaw_08d-v1-v1, origin xyz=-0.03955703826381589 -0.003868250000000062 -0.011052701243913141 rpy=-0.7853981633974496 -9.813077866773746e-17 -1.5707963267948977, axis -0.37100000000000005 0.376637 -0.848825
- added joint STS3215_03a-v2_Revolute-2: type continuous, parent STS3215_03a-v2, child Rotation_Pitch_08i-v1, origin xyz=0.012500000386367267 9.58806177834247e-11 0.018700000000000036 rpy=0.0 -0.0 1.5707963267948983, axis 0.0 0.0 1.0
- added joint STS3215_03a-v2_Revolute-4: type continuous, parent STS3215_03a-v2, child SO_ARM100_08k-1-v1, origin xyz=0.012500000670229827 2.1748424439138605e-09 -0.01769999647770381 rpy=-1.5707963267948821 0.8290313725909925 1.570796326794906, axis 0.737277 0.67559 3.750277866033529e-17
- added joint STS3215_03a-v2_Revolute-7: type continuous, parent STS3215_03a-v2, child Wrist_Roll_Pitch_08i-v1, origin xyz=0.015315395479346936 0.017378339999999878 -0.027956300980211887 rpy=-3.389728535365244e-16 -0.785398163397447 3.2517679528326754e-17, axis 0.737277 0.67559 -3.39776747869228e-17
- added joint STS3215_03a-v2_Revolute-9: type continuous, parent STS3215_03a-v2, child SO_ARM100_08k_elbow_rotate-v1, origin xyz=0.01767294000817094 -0.008673965731082376 0.02087761055724533 rpy=-0.785398163397447 4.338581489281525e-17 -3.141592652647789, axis -0.37652300000000005 -0.41090299999999996 0.830295
- joint SO_ARM100_08k-1-v1_Rigid-5: origin xyz=-0.004712700000000003 -0.12015728000000002 0.007200000000000007 rpy=4.278299853230853e-16 0.7853981633974477 2.608881203934407e-16 -> xyz=0.07447060999999999 -0.08824607999999999 -0.034330419999999987 rpy=-1.0182257570545803e-15 0.7853981633974451 -3.9257550043977953e-16
- joint SO_ARM100_08k_elbow_rotate-v1_Rigid-12: origin xyz=-0.010255080000000001 -0.04415426 -0.007413869999999996 rpy=-3.1415926535897927 0.7853981633974477 -3.12183824489694 -> xyz=-0.02753993 -0.012037259999999996 0.03473309000000001 rpy=3.1415926535897922 0.7853981633974506 -3.1218382448969435
- joint Wrist_Roll_08c-v1-v2_Rigid-17: origin xyz=-0.015 -0.022387499999999998 0.004537499999999995 rpy=1.7882708017873474e-25 -0.7853981633974491 1.5707963267948966 -> xyz=-0.023070509999999995 -0.0021048899999999995 0.014495179999999977 rpy=-1.103971260012025e-15 -0.7853981633974496 1.5707963267948926
- joint Wrist_Roll_Pitch_08i-v1_Rigid-8: origin xyz=-0.0108 0.03231723000000001 -0.004682769999999987 rpy=2.3561944901923457 6.660976308101158e-10 -3.1415926529236957 -> xyz=-0.017504029999999997 0.0031162699999999965 -0.029442650000000015 rpy=2.3561944901923457 6.660975083332575e-10 -3.1415926529236957
